File: ActionPCB.kicad_pcb (KiCad board)
At the start: 2 copper layers, 43 x 30 mm, 36 parts, among them P1 VCC, P10 GND, P11 SCL, P12 SDA, P13 CH1, P14 CH2, P15 CH3, P16 CH4, P2 GND, P3 SCL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

Commit message: Everything
Parts:
- removed C1: 10n, Capacitor_SMD:C_0603_1608Metric
- removed C2, C5: 0.1u, Capacitor_SMD:C_0603_1608Metric
- removed C3: 2.2n, Capacitor_SMD:C_0603_1608Metric
- removed C4: 0.33u, Capacitor_SMD:C_0603_1608Metric
- removed D1: Power, LED_SMD:LED_0603_1608Metric
- removed D2: Selector, LED_SMD:LED_0603_1608Metric
- removed JP1: Jumper, Jumper:SolderJumper-2_P1.3mm_Open_TrianglePad1.0x1.5mm
- removed R3, R4: 68, Resistor_SMD:R_0603_1608Metric
- removed U1: MPU-6050, Sensor_Motion:InvenSense_QFN-24_4x4mm_P0.5mm
- removed U2: AMS1117-3.3, Package_TO_SOT_SMD:SOT-223-3_TabPin2
- added J1: Conn_01x08_Male, Connector_PinHeader_2.54mm:PinHeader_1x08_P2.54mm_Vertical, F.Cu at (135.3, 57.6)
- moved JP3 13.4 mm to (124.4, 42.7), turned to 90 degrees
- moved JP2 13.1 mm to (128.2, 42.7), turned to 90 degrees
- moved R1 10.0 mm to (128.2, 50.0), turned to 0 degrees
- moved R2 7.22 mm to (128.2, 52.6), turned to 0 degrees
Connections:
- P1 pad 1: VCC -> +3V3
- P9 pad 1: VCC -> +3V3
Routing:
- net VCC: track 37.6 -> 0.00 mm
- net /SDA: track 36.0 -> 52.0 mm, vias 2 -> 3
- net Net-(JP1-Pad2): track 15.1 -> 0.00 mm, vias 2 -> 0
- net /AD0: track 38.2 -> 29.1 mm, vias 2 -> 0
- net Net-(C3-Pad1): track 8.72 -> 0.00 mm
- net +3V3: track 50.0 -> 57.8 mm, vias 2 -> 0
- net Net-(C1-Pad1): track 4.15 -> 0.00 mm
- net Net-(C2-Pad1): track 4.03 -> 0.00 mm
- net /CH3: track 33.9 -> 36.7 mm
- net Net-(D2-Pad1): track 1.80 -> 0.00 mm
- net Net-(D1-Pad1): track 1.78 -> 0.00 mm
- net /CH2: track 31.8 -> 33.5 mm
- net /SCL: track 35.9 -> 37.6 mm, vias 2 -> 3
- net /CH1: track 32.7 -> 32.1 mm
- net /CH4: track 35.4 -> 36.0 mm
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Other:
- board text added: "Action Node v0.4 16 / 03 / 22"
- board text removed: "Action Node v0.3 07 / 03 / 22"
