File: ActionPCB.kicad_sch (KiCad schematic)
At the start: 36 parts, among them P1 VCC, P10 GND, P11 SCL, P12 SDA, P13 CH1, P14 CH2, P15 CH3, P16 CH4, P2 GND, P3 SCL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

Commit message: Final board single
Parts:
- P1, P10, P11, P12, P13, P14, P15, P16, P2, P3, P4, P5, P6, P7, P8, P9: footprint TestPoint:TestPoint_Pad_D1.0mm -> Connector_Wire:SolderWirePad_1x01_SMD_1x2mm

Commit message: Everything
Parts:
- removed C1: 10n, Capacitor_SMD:C_0603_1608Metric, symbol Device:C
- removed C2, C5: 0.1u, Capacitor_SMD:C_0603_1608Metric, symbol Device:C
- removed C3: 2.2n, Capacitor_SMD:C_0603_1608Metric, symbol Device:C
- removed C4: 0.33u, Capacitor_SMD:C_0603_1608Metric, symbol Device:C
- removed D1: Power, LED_SMD:LED_0603_1608Metric, symbol Device:LED
- removed D2: Selector, LED_SMD:LED_0603_1608Metric, symbol Device:LED
- removed JP1: Jumper, Jumper:SolderJumper-2_P1.3mm_Open_TrianglePad1.0x1.5mm, symbol Jumper:SolderJumper_2_Open
- removed R3, R4: 68, Resistor_SMD:R_0603_1608Metric, symbol Device:R_Small_US
- removed U1: MPU-6050, Sensor_Motion:InvenSense_QFN-24_4x4mm_P0.5mm, symbol Sensor_Motion:MPU-6050
- removed U2: AMS1117-3.3, Package_TO_SOT_SMD:SOT-223-3_TabPin2, symbol Regulator_Linear:AMS1117-3.3
- added J1: Conn_01x08_Male, Connector_PinHeader_2.54mm:PinHeader_1x08_P2.54mm_Vertical, symbol Connector:Conn_01x08_Male
Connections:
- net VCC is gone; now on net +3V3: P1.1, P9.1
- net +3V3: now also J1.1 (Pin_1)
- net AD0: now also J1.7 (Pin_7)
- net GND: now also J1.2 (Pin_2)
- net INT: now also J1.8 (Pin_8)
- net SCL: now also J1.3 (Pin_3)
- net SDA: now also J1.4 (Pin_4)
Other:
- note added: "MPU6050"
- note removed: "MPU6050 IC"
- note removed: "Power Regulator"
- note removed: "Status LEDs"
